Commit message: Task 1-15 : iiwa : Modified Xacro to add Vacuum Gripper
 Made link and joints for the vacuum gripper and then added vacuum gripper plugin

File: iiwa_description/urdf/iiwa7.urdf.xacro (robot description, xacro)
@@ -9,4 +9,5 @@
   <xacro:arg name="origin_xyz" default="0 0 0"/>
   <xacro:arg name="origin_rpy" default="0 0 0"/>
+  <xacro:property name="link" value="0.1" /> <!-- Size of square 'camera' box -->
   <!-- Fix to world just for testing -->
   <link name="world"/>
@@ -15,3 +16,42 @@
     <origin xyz="$(arg origin_xyz)" rpy="$(arg origin_rpy)" />
   </xacro:iiwa7>
+  <!--Gripper Link-->
+  <link name="iiwa_gripper_link">
+    <!--<collision>
+      <origin xyz="0 0 0" rpy="0 0 0"/>
+      <geometry>
+        <box size="${camera_link} ${camera_link} ${camera_link}"/>
+      </geometry>
+    </collision>-->
+    <visual>
+      <origin xyz="0 0 0" rpy="0 0 0"/>
+      <geometry>
+        <box size="${link} ${link} ${link}"/>
+      </geometry>
+      <material name="red"/>
+    </visual>
+    <inertial>
+      <mass value="1e-5" />
+      <origin xyz="0 0 0" rpy="0 0 0"/>
+      <inertia ixx="1e-6" ixy="0" ixz="0" iyy="1e-6" iyz="0" izz="1e-6" />
+    </inertial>
+  </link>
+  <!--**********************************-->
+  <joint name="iiwa_gripper_joint" type="revolute">
+    <origin xyz="0 0 00.100001" rpy="0 -1.57 0"/>
+    <axis xyz="0 0 1"/>
+    <limit effort="1000.0" lower="0" upper="0" velocity="0"/>
+    <parent link="iiwa_link_7"/>
+    <child link="iiwa_gripper_link"/>
+  </joint>
+  <!--**********************************-->
+  <gazebo>
+      <plugin name="gazebo_ros_vacuum_gripper" filename="libgazebo_ros_vacuum_gripper.so">
+        <robotNamespace>/robot/left_vacuum_gripper</robotNamespace>
+        <bodyName>iiwa_gripper_link</bodyName>
+        <topicName>grasping</topicName>
+        <maxForce>500</maxForce>
+      </plugin>
+    </gazebo>
+<!--**********************************-->
 </robot>

Commit message: Task: 2-19 iiwa stack updated
The iiwa_stack package has been updated to remove the visualization of the kuka gripper.

File: iiwa_description/urdf/iiwa7.urdf.xacro (robot description, xacro)
@@ -24,5 +24,5 @@
       </geometry>
     </collision>-->
-    <visual>
+<!--     <visual>
       <origin xyz="0 0 0" rpy="0 0 0"/>
       <geometry>
@@ -31,4 +31,5 @@
       <material name="red"/>
     </visual>
+ -->
     <inertial>
       <mass value="1e-5" />
